Commit message: Fix Weichai F1 v1.1 collision geometry

File: resources/robots/weichai_f1_12/urdf/weichai_f1_12.urdf (robot description, URDF)
Before this commit: robot X1_12DOF, 48 links, 47 joints
Links:
- link left_knee_pitch_link: geometry collision mesh filename=../meshes/collision/v1_1/left_knee_pitch_collision.stl scale=1 1 1; visual mesh filename=../meshes/mujoco_stl/left_knee_pitch_bf14b2f4adf6_exact_ful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 scale=0.001 0.001 0.001
- link right_knee_pitch_link: geometry collision mesh filename=../meshes/collision/v1_1/right_knee_pitch_collision.stl scale=1 1 1; visual mesh filename=../meshes/mujoco_stl/right_knee_pitch_669ca5ac96b8_exact_fu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 scale=0.001 0.001 0.001
